File: Board/smd/Tamagotchi-Atmega8/Tamagotchi-Atmega8.kicad_pcb (KiCad board)
At the start: 2 copper layers, 47.8 x 47.8 mm, 27 parts, among them J1 Conn_02x05_Odd_Even, J2 Conn_01x02, J3 Conn_01x04, J4 Conn_01x07, J5 Conn_01x02, Q1 Q_NPN_BEC, SW1 SW_Push, U1 AMS1117, U2 ATmega328-AU, U3 DS1307Z+, X1 8MHz, X2 32768kHz

Commit message: a
Other:
- board text added: "+ (vcc)"
- board text added: "-"
- board text added: "GND"
- board text added: "SCL"
- board text added: "SDA"
- board text added: "SPEAKER"
- board text added: "VBAT"
- board text added: "VCC"
- board text added: "buttons....."
- board text added: "key"
- board text added: "usbasp"

Commit message: Board enhancement
Parts:
- SW1: footprint Button_Switch_SMD:SW_SPST_Panasonic_EVQPL_3PL_5PL_PT_A15 -> Button_Switch_SMD:SW_SPST_B3S-1000
- X1: footprint Crystal:Crystal_SMD_0603-2Pin_6.0x3.5mm_HandSoldering -> Crystal:Crystal_SMD_3225-4Pin_3.2x2.5mm
- X2: footprint Crystal:Crystal_C38-LF_D3.0mm_L8.0mm_Horizontal_1EP_style2 -> Crystal:Crystal_AT310_D3.0mm_L10.0mm_Horizontal_1EP_style2
- moved C3 3.63 mm to (117.3, 91.2), turned to 0 degrees
- moved C2 3.56 mm to (117.3, 85.1), turned to 0 degrees
- moved J5 2.17 mm to (114.3, 99.3)
- moved SW1 2.05 mm to (113.8, 75.4), turned to 180 degrees
- moved X2 0.57 mm to (123.4, 79.5)
- moved X1 0.47 mm to (117.6, 88.1), turned to 90 degrees
- turned R3 to 180 degrees
Connections:
- X1 pad 1: Net-(C2-Pad2) -> Net-(C3-Pad2)
- X1 pad 2: Net-(C3-Pad2) -> Net-(C2-Pad2)
Routing:
- net GND: track 81.1 -> 90.1 mm, vias 11 -> 9
- net Net-(C3-Pad2): track 10.9 -> 6.87 mm
- net VCC: track 180.0 -> 183.7 mm
- net Net-(C2-Pad2): track 10.7 -> 6.97 mm
- net USBASP_NRST: track 55.9 -> 54.9 mm
- net Net-(J5-Pad2): track 11.3 -> 12.2 mm
